File: Power_Distribution_Antispark.kicad_pcb (KiCad board)
At the start: 2 copper layers, 131 parts, among them J1 STM Signal Conn, J10 CSense12V_2 Conn, J11 CSense12V_3 Conn, J2 +48V Battery Conn, J3 Motor Conn, J4 CSense3V3STM Conn, J5 CSense3V3_2 Conn, J6 CSense5V_1 Conn, J7 CSense5V_2 Conn, J8 CSense5V_3 Conn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

Commit message: different layout
Parts:
- moved TP2 37.6 mm to (194.5, 116.0)
- moved R1 9.51 mm to (184.5, 96.5)
- moved R8 7.01 mm to (185.5, 99.5)
- moved R21 7.00 mm to (197.6, 91.6), turned to 90 degrees
- moved C23 6.52 mm to (204.4, 91.3), turned to -90 degrees
- moved J3 6.00 mm to (212.7, 114.8)
- moved D9 5.41 mm to (177.5, 74.0)
- moved R2 4.21 mm to (180.5, 93.5), turned to -90 degrees
- moved J2 3.97 mm to (212.8, 62.2)
- moved F2 3.25 mm to (179.0, 104.0)
- moved D3 3.02 mm to (186.0, 87.5)
- moved R3 3.02 mm to (186.0, 90.0)
- moved R4 3.02 mm to (185.9, 85.4)
- moved R12 2.73 mm to (182.5, 101.0), turned to 180 degrees
- moved R6 2.56 mm to (183.0, 104.0)
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