File: CSense.kicad_sch (KiCad schematic)
At the start: 4 parts, among them J10 ${SHEETNAME} Conn, U13 INA181A3IDBVR

Commit message: final schematic
Connections:
- net +5V_PC renamed +5V
Changed lines of the file:
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@@
 			)
 		)
-		(property "Value" "+5V_PC"
+		(property "Value" "+5V"
 			(at 151.13 64.77 0)
 			(effects

Commit message: final schematic
Parts:
- removed C37: 1uF, Capacitor_SMD:C_0201_0603Metric, symbol Device:C_Small
- added C24: 1uF, Capacitor_SMD:C_0603_1608Metric, symbol Device:C_Small
- renumbered J10 to J4, R37 to R39, U13 to U7
Connections:
- net +5V: now also C24.1
- net GND: now also C24.2

Commit message: fixed connectors
Parts:
- J4: footprint CustomFootprintLibrary:M20-9990246 -> CustomFootprintLibrary:CONN_B2B-ZR_02P_JST
Changed lines of the file:
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@@
 			)
 		)
-		(property "Footprint" "CustomFootprintLibrary:M20-9990246"
+		(property "Footprint" "CustomFootprintLibrary:CONN_B2B-ZR_02P_JST"
 			(at 134.62 102.87 0)
 			(effects
@@
 			)
 		)
-		(property "Datasheet" "https://www.digikey.ca/en/products/detail/harwin-inc/M20-9990246/3728226"
+		(property "Datasheet" "https://www.digikey.ca/en/products/detail/jst-sales-america-inc/B2B-ZR/926564"
 			(at 134.62 102.87 0)
 			(effects
@@
 			)
 		)
-		(property "Description" "CONN HEADER VERT 2POS 2.54MM"
+		(property "Description" "CONN HEADER VERT 2POS 1.5MM"
 			(at 134.62 102.87 0)
 			(effects
